Commit message: added mesh to wheels, needs fixing so it works in gazebo and rviz

File: description/robot_core.xacro (robot description, xacro)
@@ -41,7 +41,8 @@
     <!-- Front Left Wheel -->
     <link name="front_left_wheel">
-        <visual>
+        <visual name='front_left_wheel_visual'>
+            <origin xyz="0 0 0" rpy="1.5708 0 0" />
             <geometry>
-                <cylinder radius="0.0485" length="0.045" />
+                <mesh filename="$(find gulliverkli)/meshes/mecanum_wheel_left.stl" scale="1 1 1" />
             </geometry>
             <material name="grey" />
@@ -67,7 +68,8 @@
     <!-- Front Right Wheel -->
     <link name="front_right_wheel">
-        <visual>
+        <visual name='front_right_wheel_visual'>
+            <origin xyz="0 0 0" rpy="1.5708 0 0" />
             <geometry>
-                <cylinder radius="0.0485" length="0.045" />
+                <mesh filename="$(find gulliverkli)/meshes/mecanum_wheel_right.stl" scale="1 1 1" />
             </geometry>
             <material name="grey" />
@@ -93,7 +95,8 @@
     <!-- rear Left Wheel -->
     <link name="rear_left_wheel">
-        <visual>
+        <visual name='rear_left_wheel_visual'>
+            <origin xyz="0 0 0" rpy="1.5708 0 0" />
             <geometry>
-                <cylinder radius="0.0485" length="0.045" />
+                <mesh filename="$(find gulliverkli)/meshes/mecanum_wheel_right.stl" scale="1 1 1" />
             </geometry>
             <material name="grey" />
@@ -119,7 +122,8 @@
     <!-- rear Right Wheel -->
     <link name="rear_right_wheel">
-        <visual>
+        <visual name='rear_right_wheel_visual'>
+            <origin xyz="0 0 0" rpy="1.5708 0 0" />
             <geometry>
-                <cylinder radius="0.0485" length="0.045" />
+                <mesh filename="$(find gulliverkli)/meshes/mecanum_wheel_left.stl" scale="1 1 1" />
             </geometry>
             <material name="grey" />
