Commit message: Gazebo, contorls, Rviz working

File: description/gulliverkli.urdf.xacro (robot description, xacro)
@@ -2,3 +2,4 @@
 <robot xmlns:xacro="http://www.ros.org/wiki/xacro" name="gulliverkli">
     <xacro:include filename="robot_core.xacro" />
+    <xacro:include filename="gazebo_control.xacro" />
 </robot>

File: description/robot_core.xacro (robot description, xacro)
@@ -1,5 +1,6 @@
 <?xml version="1.0"?>
-<robot xmlns:xacro="http://www.ros.org/wiki/xacro">
+<robot xmlns:xacro="http://www.ros.org/wiki/xacro" xmlns:gz="http://gazebosim.org/schema">
     <xacro:include filename="inertial_macros.xacro" />
+    <xacro:include filename="gazebo_control.xacro" />
     <!-- Material Definitions -->
     <material name="blue">
@@ -34,5 +35,5 @@
         </collision>
         <xacro:inertial_box mass="2.2" x="0.3" y="0.19" z="0.075">
-            <origin xyz="0.15 0 0.0375" rpy="0 0 0"/>
+            <origin xyz="0.15 0 0.0375" rpy="0 0 0" />
         </xacro:inertial_box>
     </link>
@@ -43,4 +44,6 @@
         <origin xyz="0.130 0.1275 0" rpy="-${pi/2} 0 0" />
         <axis xyz="0 0 1" />
+        <limit effort="10000" velocity="10" />
+        <dynamics damping="1.0" friction="1.0" />
     </joint>
     <!-- Front Left Wheel -->
@@ -58,5 +61,5 @@
         </collision>
         <xacro:inertial_cylinder mass="0.15" length="0.045" radius="0.0485">
-            <origin xyz="0 0 0" rpy="0 0 0"/>
+            <origin xyz="0 0 0" rpy="0 0 0" />
         </xacro:inertial_cylinder>
     </link>
@@ -67,4 +70,6 @@
         <origin xyz="0.130 -0.1275 0" rpy="${pi/2} 0 0" />
         <axis xyz="0 0 -1" />
+        <limit effort="10000" velocity="10" />
+        <dynamics damping="1.0" friction="1.0" />
     </joint>
     <!-- Front Right Wheel -->
@@ -82,5 +87,5 @@
         </collision>
         <xacro:inertial_cylinder mass="0.15" length="0.045" radius="0.0485">
-            <origin xyz="0 0 0" rpy="0 0 0"/>
+            <origin xyz="0 0 0" rpy="0 0 0" />
         </xacro:inertial_cylinder>
     </link>
@@ -91,4 +96,6 @@
         <origin xyz="-0.130 0.1275 0" rpy="-${pi/2} 0 0" />
         <axis xyz="0 0 1" />
+        <limit effort="10000" velocity="10" />
+        <dynamics damping="1.0" friction="1.0" />
     </joint>
     <!-- rear Left Wheel -->
@@ -106,5 +113,5 @@
         </collision>
         <xacro:inertial_cylinder mass="0.15" length="0.045" radius="0.0485">
-            <origin xyz="0 0 0" rpy="0 0 0"/>
+            <origin xyz="0 0 0" rpy="0 0 0" />
         </xacro:inertial_cylinder>
     </link>
@@ -115,4 +122,6 @@
         <origin xyz="-0.130 -0.1275 0" rpy="${pi/2} 0 0" />
         <axis xyz="0 0 -1" />
+        <limit effort="10000" velocity="10" />
+        <dynamics damping="1.0" friction="1.0" />
     </joint>
     <!-- rear Right Wheel -->
@@ -130,6 +139,64 @@
         </collision>
         <xacro:inertial_cylinder mass="0.15" length="0.045" radius="0.0485">
-            <origin xyz="0 0 0" rpy="0 0 0"/>
-        </xacro:inertial_cylinder>
-    </link>
+            <origin xyz="0 0 0" rpy="0 0 0" />
+        </xacro:inertial_cylinder>
+    </link>
+    <!-- STEP 4 - Gazebo frictions -->
+    <gazebo reference='front_left_wheel'>
+        <collision>
+            <surface>
+                <friction>
+                    <ode>
+                        <mu>1.5</mu>
+                        <mu2>0.0</mu2>
+                        <fdir1 gz:expressed_in="base_link">1 -1 0</fdir1>
+                    </ode>
+                </friction>
+            </surface>
+        </collision>
+    </gazebo>
+    <gazebo reference='rear_left_wheel'>
+        <collision>
+            <surface>
+                <friction>
+                    <ode>
+                        <mu>1.5</mu>
+                        <mu2>0.0</mu2>
+                        <fdir1 gz:expressed_in="base_link">1 1 0</fdir1>
+                    </ode>
+                </friction>
+            </surface>
+        </collision>
+    </gazebo>
+    <gazebo reference='front_right_wheel'>
+        <collision>
+            <surface>
+                <friction>
+                    <ode>
+                        <mu>1.5</mu>
+                        <mu2>0.0</mu2>
+                        <fdir1 gz:expressed_in="base_link">1 1 0</fdir1>
+                    </ode>
+                </friction>
+            </surface>
+        </collision>
+    </gazebo>
+    <gazebo reference='rear_right_wheel'>
+        <collision>
+            <surface>
+                <friction>
+                    <ode>
+                        <mu>1.5</mu>
+                        <mu2>0.0</mu2>
+                        <fdir1 gz:expressed_in="base_link">1 -1 0</fdir1>
+                    </ode>
+                </friction>
+            </surface>
+        </collision>
+    </gazebo>
+    <gazebo reference="base_link">
+        <mu1>0.000002</mu1>
+        <mu2>0.000002</mu2>
+        <!-- <material>Gazebo/Red</material> -->
+    </gazebo>
 </robot>

Commit message: added gz_bridge.yaml, adjusted URDF

File: description/gulliverkli.urdf.xacro (robot description, xacro)
@@ -1,5 +1,7 @@
 <?xml version="1.0"?>
 <robot xmlns:xacro="http://www.ros.org/wiki/xacro" name="gulliverkli">
+    <xacro:include filename="materials.xacro" />
     <xacro:include filename="robot_core.xacro" />
     <xacro:include filename="gazebo_control.xacro" />
+    <xacro:include filename="lidar.xacro" />
 </robot>

File: description/robot_core.xacro (robot description, xacro)
@@ -2,12 +2,4 @@
 <robot xmlns:xacro="http://www.ros.org/wiki/xacro" xmlns:gz="http://gazebosim.org/schema">
     <xacro:include filename="inertial_macros.xacro" />
-    <xacro:include filename="gazebo_control.xacro" />
-    <!-- Material Definitions -->
-    <material name="blue">
-        <color rgba="0.1 0.1 1 1" /> <!-- Blue -->
-    </material>
-    <material name="grey">
-        <color rgba="0.2 0.2 0.2 1" /> <!-- grey -->
-    </material>
     <!-- Base Link -->
     <link name="base_link">
@@ -26,5 +18,5 @@
                 <box size="0.3 0.19 0.075" />
             </geometry>
-            <material name="blue" />
+            <material name="orange" />
         </visual>
         <collision>

Commit message: FINALLY FIXED THE DAMN MESH PROBLEM

File: description/gulliverkli.urdf.xacro (robot description, xacro)
@@ -5,3 +5,5 @@
     <xacro:include filename="gazebo_control.xacro" />
     <xacro:include filename="lidar.xacro" />
+    <!-- <xacro:include filename="camera_kinect.xacro" /> -->
+    <!-- <xacro:include filename="depth_kinect.xacro" /> -->
 </robot>

File: description/lidar.xacro (robot description, xacro)
@@ -41,5 +41,5 @@
             </lidar>
             <topic>scan</topic>
-            <gz_frame_id>laser_frame</gz_frame_id>
+            <!-- <gz_frame_id>laser_frame</gz_frame_id> -->
         </sensor>
     </gazebo>

File: description/robot_core.xacro (robot description, xacro)
@@ -44,5 +44,5 @@
             <origin xyz="0 0 0" rpy="1.5708 0 0" />
             <geometry>
-                <mesh filename="$(find gulliverkli)/meshes/mecanum_wheel_left.stl" scale="1 1 1" />
+                <mesh filename="package://gulliverkli/meshes/mecanum_wheel_left.stl" scale="1 1 1" />
             </geometry>
             <material name="grey" />
@@ -71,5 +71,5 @@
             <origin xyz="0 0 0" rpy="1.5708 0 0" />
             <geometry>
-                <mesh filename="$(find gulliverkli)/meshes/mecanum_wheel_right.stl" scale="1 1 1" />
+                <mesh filename="package://gulliverkli/meshes/mecanum_wheel_right.stl" scale="1 1 1" />
             </geometry>
             <material name="grey" />
@@ -98,5 +98,5 @@
             <origin xyz="0 0 0" rpy="1.5708 0 0" />
             <geometry>
-                <mesh filename="$(find gulliverkli)/meshes/mecanum_wheel_right.stl" scale="1 1 1" />
+                <mesh filename="package://gulliverkli/meshes/mecanum_wheel_right.stl" scale="1 1 1" />
             </geometry>
             <material name="grey" />
@@ -125,5 +125,5 @@
             <origin xyz="0 0 0" rpy="1.5708 0 0" />
             <geometry>
-                <mesh filename="$(find gulliverkli)/meshes/mecanum_wheel_left.stl" scale="1 1 1" />
+                <mesh filename="package://gulliverkli/meshes/mecanum_wheel_left.stl" scale="1 1 1" />
             </geometry>
             <material name="grey" />
